File: Hardware/PCB_DIY_V4/Alita_PCB_V4.kicad_pcb (KiCad board)
At the start: 2 copper layers, 100 x 55 mm, 30 parts, among them J1 Interface, J2 Vss, J4 Conn_01x03_Pin, J5 Driver, J6 MUX_header1, J7 MUX_header2, P1 5v_Pins, P2 3.3v_Pins, U1 MUX 4067, U2 ESP32_NODEMCU

Commit message: Añadi el simbolo arreglado al esquematico y PCB
Parts:
- added U3: ~, MixLib:Nodemcu_ESP32S_38pin, F.Cu at (124.6, 73.2)
Connections:
- U2 pad 16: /P13 -> unconnected-(U2-GPIO13-Pad16)
