File: Hardware/PCB_DIY_V4/Alita_PCB_V4.kicad_sch (KiCad schematic)
At the start: 32 parts, among them J1 VS, J2 Conn_01x08_Pin, J3 Conn_01x08_Pin, J4 ESC, J5 Driver In, J6 Oled SSD1306, J7 Boton1, J8 Boton2, P1 Multiplexor 5v, P2 Multiplexor 3v3, U2 CD74HC4067SM, U3 ESP32-WROOM-32E, U4 ESP32_NODEMCU

Commit message: Avances en esquematico
Parts:
- removed C1: ~, Capacitor_SMD:C_0805_2012Metric_Pad1.18x1.45mm_HandSolder, symbol Device:C_Small
- removed C4: 100nF, Capacitor_SMD:C_0805_2012Metric_Pad1.18x1.45mm_HandSolder, symbol Device:C_Small
- removed D1, D2: LED, LED_SMD:LED_0805_2012Metric_Pad1.15x1.40mm_HandSolder, symbol Device:LED
- removed J6: Oled SSD1306, ConnectorMolex2:Molex_KK-254_AE-6410-04A_1x04_P2.54mm_Vertical, symbol EESTN5:HEADER_4
- removed J7: Boton1, Connector_PinHeader_2.54mm:PinHeader_1x02_P2.54mm_Horizontal, symbol EESTN5:HEADER_2
- removed J8: Boton2, Connector_PinHeader_2.54mm:PinHeader_1x02_P2.54mm_Horizontal, symbol EESTN5:HEADER_2
- removed Jd1: FTDI 232RL, Connector_PinHeader_2.54mm:PinHeader_1x04_P2.54mm_Vertical, symbol EESTN5:HEADER_4
- removed R1, R2: 220, Resistor_SMD:R_0805_2012Metric_Pad1.20x1.40mm_HandSolder, symbol Device:R
- removed R3, R4: 10k, Resistor_SMD:R_0805_2012Metric_Pad1.20x1.40mm_HandSolder, symbol EESTN5:R
- removed SW_BOOT1: SW_Push, EESTN5:Pulsador_SMD_2_BAJO, symbol EESTN5:SW_Push
- removed SW_EN1: SW_Push, Button_Switch_SMD:SW_Tactile_SPST_NO_Straight_CK_PTS636Sx25SMTRLFS, symbol EESTN5:SW_Push
- removed U2: CD74HC4067SM, Package_SO:SSOP-24_5.3x8.2mm_P0.65mm, symbol 74xx:CD74HC4067SM
- removed U3: ESP32-WROOM-32E, TriatlonLibrary:ESP32-WROOM-32E, symbol Librerias:ESP32-WROOM-32E
- added J6: Button1, symbol Connector:Conn_01x02_Pin
- added J7: Button2, symbol Connector:Conn_01x02_Pin
- added J9: Conn_01x04_Pin, ConnectorMolex2:Molex_KK-254_AE-6410-04A_1x04_P2.54mm_Vertical, symbol Connector:Conn_01x04_Pin
- added R1, R2: 10k, symbol Device:R_Small
- J1: value VS -> Vss
- J2: value Conn_01x08_Pin -> MUX_Header2
- J3: value Conn_01x08_Pin -> MUX_Header1
- J5: value Driver In -> Driver Input
- P1: value Multiplexor 5v -> 5v_Pins
- P2: value Multiplexor 3v3 -> 3.3v_Pins
- U1: value ~ -> MUX 4067
Connections:
- net GPIO 35 is gone; now on net ESC: J4.1 (Pin_1)
- net P16 is gone; now on net MB2: U4.27 (GPIO16)
- net P17 is gone; now on net MB1: U4.28 (GPIO17)
- net P21 is gone; now on net SDA: U4.33 (GPIO21)
- net P22 is gone; now on net SCL: U4.36 (GPIO22)
- net P25 is gone; now on net SIG: U1.17 (SIG), U4.10 (GPIO25)
- net P26 is gone; now on net MA1: U4.11 (GPIO26)
- net P27 is gone; now on net MA2: U4.12 (GPIO27)
- net P32 is gone; now on net S2: U1.19 (S2), U4.8 (GPIO32)
- net P33 is gone; now on net S3: U1.18 (S3), U4.9 (GPIO33)
- net P34 is gone; now on net S1: U4.6 (GPIO34)
- net P4 is gone; now on net S0: U1.21 (S0), U4.26 (GPIO4)
- net +3.3V: now also U1.23 (VCC), R1.1, R2.1
- net +5V: now also J9.3 (Pin_3)
- net ESC: now also U4.7 (GPIO35)
- net GND: now also U1.24 (GND), J6.2 (Pin_2), J7.2 (Pin_2), J9.4 (Pin_4)
- net P13: no longer U4.14 (GPIO12)
- net S1: now also U1.20 (S1)
- net SCL: now also J9.2 (Pin_2)
- net SDA: now also J9.1 (Pin_1)
- net P19: now reaches U4.31 (GPIO19)
- net at U1.1 (C15): now also J3.8 (Pin_8)
- net at U1.10 (C6): now also J2.7 (Pin_7)
- net at U1.11 (C5): now also J2.6 (Pin_6)
- net at U1.12 (C4): now also J2.5 (Pin_5)
- net at U1.13 (C3): now also J2.4 (Pin_4)
- net at U1.14 (C2): now also J2.3 (Pin_3)
- net at U1.15 (C1): now also J2.2 (Pin_2)
- net at U1.16 (C0): now also J2.1 (Pin_1)
- net at U1.2 (C14): now also J3.7 (Pin_7)
- net at U1.3 (C13): now also J3.6 (Pin_6)
- net at U1.4 (C12): now also J3.5 (Pin_5)
- net at U1.5 (C11): now also J3.4 (Pin_4)
- net at U1.6 (C10): now also J3.3 (Pin_3)
- net at U1.7 (C9): now also J3.2 (Pin_2)
- net at U1.8 (C8): now also J3.1 (Pin_1)
- net at U1.9 (C7): now also J2.8 (Pin_8)
- net P0: no longer names the net of U4.25 (GPIO0)
- net P1: no longer names the net of U4.35 (GPIO1)
- net P18 renamed Button2
- net Button2: now also J7.1 (Pin_1), R2.2
- net P2: no longer names the net of U4.24 (GPIO2)
- net P3: no longer names the net of U4.34 (GPIO3)
- removed net P35: U1.20 (S1), U4.7 (GPIO35)
- net P5 renamed Button1
- net Button1: now also J6.1 (Pin_1), R1.2
- new net P12: U4.14 (GPIO12)
- no-connect marks 20 -> 12
Other:
- note added: "Analog Multiplexer"
- note added: "BLDC Controller"
- note added: "ESP32"
- note added: "Holes"
- note added: "Interface Buttons"
- note added: "Motor Driver Input"
- note added: "OLED Display"
- note added: "Switching Voltage Supply"
- note added: "Voltage Breakout Pins"
- note removed: "AGUJEROS"
- note removed: "BOTONES"
- note removed: "DRIVER INPUT"
- note removed: "EN Y BOOT"
- note removed: "ESC PIN"
- note removed: "ESP32 MODULE"
- note removed: "I2C"
- note removed: "LED"
- note removed: "MULTIPLEXOR CD74HC4067"
- note removed: "POWER SUPPLY"
- note removed: "PROGRAMADOR"
- note removed: "https://www.studiopieters.nl/esp32-pinout/"
- moved on the sheet: C2, C3, D3, H1, H2, H3, H4, J1, J2, J3, J4, J5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

Commit message: Asignacion de huellas
Parts:
- removed J4: ESC, Connector_Molex:Molex_KK-254_AE-6410-02A_1x02_P2.54mm_Vertical, symbol Connector:Conn_01x02_Pin
- added D1: 1N5819, Diode_SMD:D_SMA, symbol Device:D_Small
- added J8: Conn_01x03_Pin, Connector_Molex:Molex_KK-254_AE-6410-03A_1x03_P2.54mm_Vertical, symbol Connector:Conn_01x03_Pin
- C3: footprint (none) -> Capacitor_SMD:CP_Elec_5x4.5
- D3: value M7 -> 1N5819; footprint (none) -> Diode_SMD:D_SMA
- J6, J7: footprint (none) -> Connector_Molex:Molex_KK-254_AE-6410-02A_1x02_P2.54mm_Vertical
- J9: footprint ConnectorMolex2:Molex_KK-254_AE-6410-04A_1x04_P2.54mm_Vertical -> Connector_Molex:Molex_KK-254_AE-6410-04A_1x04_P2.54mm_Vertical
- R1, R2: footprint (none) -> PCM_Resistor_SMD_AKL:R_0805_2012Metric_Pad1.15x1.40mm_HandSolder
- U1: footprint (none) -> MixLib:HP4067_module
Connections:
- net +5V: now also D1.1 (K)
- net ESC: now also J8.1 (Pin_1)
- net GND: now also J8.3 (Pin_3)
- new net: D1.2 (A), J8.2 (Pin_2)

Commit message: Primer posicionamiento de componentes en PCB
Parts:
- removed J2: MUX_Header2, Connector_PinHeader_2.54mm:PinHeader_1x08_P2.54mm_Horizontal, symbol Connector:Conn_01x08_Pin
- removed J3: MUX_Header1, Connector_PinHeader_2.54mm:PinHeader_1x08_P2.54mm_Horizontal, symbol Connector:Conn_01x08_Pin
- removed J5: Driver Input, Connector_PinHeader_2.54mm:PinHeader_1x07_P2.54mm_Horizontal, symbol Connector:Conn_01x07_Pin
- removed J6: Button1, Connector_Molex:Molex_KK-254_AE-6410-02A_1x02_P2.54mm_Vertical, symbol Connector:Conn_01x02_Pin
- removed J7: Button2, Connector_Molex:Molex_KK-254_AE-6410-02A_1x02_P2.54mm_Vertical, symbol Connector:Conn_01x02_Pin
- added J2: MUX_header, Connector_PinHeader_2.54mm:PinHeader_1x16_P2.54mm_Horizontal, symbol Connector:Conn_01x16_Pin
- added J4: Driver, Connector_PinHeader_2.54mm:PinHeader_1x06_P2.54mm_Horizontal, symbol Connector:Conn_01x06_Pin
- added J5: Buttons, Connector_Molex:Molex_KK-254_AE-6410-04A_1x04_P2.54mm_Vertical, symbol Connector:Conn_01x04_Pin
Connections:
- net +5V: now also J4.1 (Pin_1)
- net Button1: now also J5.1 (Pin_1)
- net Button2: now also J5.3 (Pin_3)
- net GND: now also J4.6 (Pin_6), J5.2 (Pin_2), J5.4 (Pin_4)
- net MA1: now also J4.5 (Pin_5)
- net MA2: now also J4.4 (Pin_4)
- net MB1: now also J4.3 (Pin_3)
- net MB2: now also J4.2 (Pin_2)
- net at U1.1 (C15): now also J2.1 (Pin_1)
- net at U1.10 (C6): now also J2.10 (Pin_10)
- net at U1.11 (C5): now also J2.11 (Pin_11)
- net at U1.12 (C4): now also J2.12 (Pin_12)
- net at U1.13 (C3): now also J2.13 (Pin_13)
- net at U1.14 (C2): now also J2.14 (Pin_14)
- net at U1.15 (C1): now also J2.15 (Pin_15)
- net at U1.16 (C0): now also J2.16 (Pin_16)
- net at U1.2 (C14): now also J2.2 (Pin_2)
- net at U1.3 (C13): now also J2.3 (Pin_3)
- net at U1.4 (C12): now also J2.4 (Pin_4)
- net at U1.5 (C11): now also J2.5 (Pin_5)
- net at U1.6 (C10): now also J2.6 (Pin_6)
- net at U1.7 (C9): now also J2.7 (Pin_7)
- net at U1.8 (C8): now also J2.8 (Pin_8)
- net at U1.9 (C7): now also J2.9 (Pin_9)
Other:
- moved on the sheet: R1, R2

Commit message: Modificacion de footprint y posicionamiento
Parts:
- removed J2: MUX_header, Connector_PinHeader_2.54mm:PinHeader_1x16_P2.54mm_Horizontal, symbol Connector:Conn_01x16_Pin
- added J2: MUX_header1, Connector_PinHeader_2.54mm:PinHeader_1x08_P2.54mm_Horizontal, symbol Connector:Conn_01x08_Pin
- added J3: MUX_header2, Connector_PinHeader_2.54mm:PinHeader_1x08_P2.54mm_Horizontal, symbol Connector:Conn_01x08_Pin
Connections:
- net at U1.1 (C15): now also J3.1 (Pin_1)
- net at U1.10 (C6): now also J2.2 (Pin_2)
- net at U1.11 (C5): now also J2.3 (Pin_3)
- net at U1.12 (C4): now also J2.4 (Pin_4)
- net at U1.13 (C3): now also J2.5 (Pin_5)
- net at U1.14 (C2): now also J2.6 (Pin_6)
- net at U1.15 (C1): now also J2.7 (Pin_7)
- net at U1.16 (C0): now also J2.8 (Pin_8)
- net at U1.2 (C14): now also J3.2 (Pin_2)
- net at U1.3 (C13): now also J3.3 (Pin_3)
- net at U1.4 (C12): now also J3.4 (Pin_4)
- net at U1.5 (C11): now also J3.5 (Pin_5)
- net at U1.6 (C10): now also J3.6 (Pin_6)
- net at U1.7 (C9): now also J3.7 (Pin_7)
- net at U1.8 (C8): now also J3.8 (Pin_8)
- net at U1.9 (C7): now also J2.1 (Pin_1)
Changed lines of the file:
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@@
+	)
+	(symbol
+		(lib_id "Connector:Conn_01x08_Pin")
+		(at 118.11 45.72 0)
+		(unit 1)
+		(exclude_from_sim no)
+		(in_bom yes)
+		(on_board yes)
+		(dnp no)
+		(property "Reference" "J3"
+			(at 109.982 42.164 0)
+			(effects
+				(font
+					(size 1.27 1.27)
+				)
+			)
+		)
+		(property "Value" "MUX_header2"
+			(at 109.982 44.704 0)
+			(effects
+				(font
+					(size 1.27 1.27)
+				)
+			)
+		)
+		(property "Footprint" "Connector_PinHeader_2.54mm:PinHeader_1x08_P2.54mm_Horizontal"
+			(at 118.11 45.72 0)
+			(effects
+				(font
+					(size 1.27 1.27)
+				)
+				(hide yes)
+			)
+		)
+		(property "Datasheet" "~"
+			(at 118.11 45.72 0)
+			(effects
+				(font
+					(size 1.27 1.27)
+				)
+				(hide yes)
+			)
+		)
+		(property "Description" "Generic connector, single row, 01x08, script generated"
+			(at 118.11 45.72 0)
+			(effects
+				(font
+					(size 1.27 1.27)
+				)
+				(hide yes)
+			)
+		)
+		(pin "3"
+		)
+		(pin "4"
+		)
+		(pin "7"
+		)
+		(pin "1"
+		)
+		(pin "2"
+		)
+		(pin "5"
+		)
+		(pin "8"
+		)
+		(pin "6"
+		)
+		(instances
+			(project "Alita_PCB_V4"
+				(path "/65967704-c20e-4a94-b405-935304512286"
+					(reference "J3")
+					(unit 1)
+				)
+			)
+		)
 	)
 	(symbol
@@
 	)
 	(symbol
-		(lib_id "Connector:Conn_01x16_Pin")
-		(at 118.11 55.88 0)
-		(unit 1)
-		(exclude_from_sim no)
-		(in_bom yes)
-		(on_board yes)
-		(dnp no)
-		(fields_autoplaced yes)
-		(property "Reference" "J2"
-			(at 118.745 33.02 0)
-			(effects
-				(font
-					(size 1.27 1.27)
-				)
-			)
-		)
-		(property "Value" "MUX_header"
-			(at 118.745 35.56 0)
-			(effects
-				(font
-					(size 1.27 1.27)
-				)
-			)
-		)
-		(property "Footprint" "Connector_PinHeader_2.54mm:PinHeader_1x16_P2.54mm_Horizontal"
-			(at 118.11 55.88 0)
-			(effects
-				(font
-					(size 1.27 1.27)
-				)
-				(hide yes)
-			)
-		)
-		(property "Datasheet" "~"
-			(at 118.11 55.88 0)
-			(effects
-				(font
-					(size 1.27 1.27)
-				)
-				(hide yes)
-			)
-		)
-		(property "Description" "Generic connector, single row, 01x16, script generated"
-			(at 118.11 55.88 0)
-			(effects
-				(font
-					(size 1.27 1.27)
-				)
-				(hide yes)
-			)
-		)
-		(pin "5"
-		)
-		(pin "11"
-		)
-		(pin "3"
-		)
-		(pin "8"
-		)
-		(pin "16"
-		)
-		(pin "6"
-		)
-		(pin "9"
-		)
-		(pin "12"
-		)
-		(pin "13"
-		)
-		(pin "14"
-		)
-		(pin "2"
-		)
-		(pin "10"
-		)
-		(pin "7"
-		)
-		(pin "15"
-		)
-		(pin "4"
-		)
-		(pin "1"
-		)
-		(instances
-			(project ""
-				(path "/65967704-c20e-4a94-b405-935304512286"
-					(reference "J2")
-					(unit 1)
-				)
-			)
-		)
-	)
-	(symbol
 		(lib_name "GND_3")
 		(lib_id "power:GND")
@@
 					(unit 1)
 				)
+			)
+		)
+	)
+	(symbol
+		(lib_id "Connector:Conn_01x08_Pin")
+		(at 118.11 66.04 0)
+		(unit 1)
+		(exclude_from_sim no)
+		(in_bom yes)
+		(on_board yes)
+		(dnp no)
+		(property "Reference" "J2"
+			(at 109.982 62.484 0)
+			(effects
+				(font
+					(size 1.27 1.27)
+				)
+			)
+		)
+		(property "Value" "MUX_header1"
+			(at 109.982 65.024 0)
+			(effects
+				(font
+					(size 1.27 1.27)
+				)
+			)
+		)
+		(property "Footprint" "Connector_PinHeader_2.54mm:PinHeader_1x08_P2.54mm_Horizontal"
+			(at 118.11 66.04 0)
+			(effects
+				(font
+					(size 1.27 1.27)
+				)
+				(hide yes)
+			)
+		)
+		(property "Datasheet" "~"
+			(at 118.11 66.04 0)
+			(effects
+				(font
+					(size 1.27 1.27)
+				)
+				(hide yes)
+			)
+		)
+		(property "Description" "Generic connector, single row, 01x08, script generated"
+			(at 118.11 66.04 0)
+			(effects
+				(font
+					(size 1.27 1.27)
+				)
+				(hide yes)
+			)
+		)
+		(pin "3"
+		)
+		(pin "4"
+		)
+		(pin "7"
+		)
+		(pin "1"
+		)
+		(pin "2"
+		)
+		(pin "5"
+		)
+		(pin "8"
+		)
+		(pin "6"
+		)
+		(instances
+			(project ""
+				(path "/65967704-c20e-4a94-b405-935304512286"
+					(reference "J2")
+					(unit 1)
+				)
