File: Hardware/PCB_DIY_V4/PCB_DIY_V4.kicad_sch (KiCad schematic)
At the start: 22 parts, among them J1 Interface, J2 Vss, J4 Conn_01x03_Pin, J5 Driver, J6 MUX_header1, J7 MUX_header2, P1 5v_Pins, P2 3.3v_Pins, U1 MUX 4067, U2 ESP32_NODEMCU

Commit message: Arregle la PCB
Arregle la PCB lol
Parts:
- removed U2: ESP32_NODEMCU, MixLib:Nodemcu_ESP32S_38pin, symbol MacroLib:ESP32_NODEMCU
Connections:
- net +5V: now also U3.19 (5V)
- net GND: now also U3.32 (GND); no longer U3.15 (GPIO13)
- net MA2: now also U3.10 (GPIO26); no longer U3.11 (GPIO27)
Other:
- moved on the sheet: U3
